File: hardware/ir_converter.kicad_pcb (KiCad board)
At the start: 2 copper layers, 37.3 x 52.1 mm, 46 parts, among them J1 MX-47346-0001, J2 SWD, J3 TP, J4 TP, Q1 LL-S350PTC-1A, Q2 BC817-40, SW1 RESET, SW2 SW2, U1 TLV70033DDCT, U2 USBLC6-2, U3 STM32F103C8T6

Commit message: New PCB is ready.
Parts:
- added C11: 1uF, Capacitors_SMD:C_0603_HandSoldering, F.Cu at (106.6, 114.3)
- added REF**: VIA_03_30mil, CustomFootprints:VIA_03_30mil, F.Cu at (94.2, 112.0)
- added REF**: VIA_03_30mil, CustomFootprints:VIA_03_30mil, F.Cu at (83.6, 122.8)
- added REF**: VIA_03_30mil, CustomFootprints:VIA_03_30mil, F.Cu at (82.4, 120.7)
- added REF**: VIA_03_30mil, CustomFootprints:VIA_03_30mil, F.Cu at (82.4, 118.6)
- added REF**: VIA_03_30mil, CustomFootprints:VIA_03_30mil, F.Cu at (82.4, 117.0)
- added REF**: VIA_03_30mil, CustomFootprints:VIA_03_30mil, F.Cu at (82.4, 122.8)
- added REF**: VIA_03_30mil, CustomFootprints:VIA_03_30mil, F.Cu at (82.4, 114.8)
- added REF**: VIA_03_30mil, CustomFootprints:VIA_03_30mil, F.Cu at (82.4, 107.6)
- added REF**: VIA_03_30mil, CustomFootprints:VIA_03_30mil, F.Cu at (82.4, 99.9)
- added REF**: VIA_03_30mil, CustomFootprints:VIA_03_30mil, F.Cu at (82.4, 92.3)
- added REF**: VIA_03_30mil, CustomFootprints:VIA_03_30mil, F.Cu at (101.7, 98.8)
- added REF**: VIA_03_30mil, CustomFootprints:VIA_03_30mil, F.Cu at (97.8, 112.0)
- added REF**: VIA_03_30mil, CustomFootprints:VIA_03_30mil, F.Cu at (103.5, 98.8)
- added REF**: VIA_03_30mil, CustomFootprints:VIA_03_30mil, F.Cu at (103.5, 96.6)
- added REF**: VIA_03_30mil, CustomFootprints:VIA_03_30mil, F.Cu at (101.7, 96.6)
- added REF**: VIA_03_30mil, CustomFootprints:VIA_03_30mil, F.Cu at (101.9, 93.6)
- added REF**: VIA_03_30mil, CustomFootprints:VIA_03_30mil, F.Cu at (103.3, 93.6)
- added REF**: VIA_03_30mil, CustomFootprints:VIA_03_30mil, F.Cu at (106.6, 92.1)
- added REF**: VIA_03_30mil, CustomFootprints:VIA_03_30mil, F.Cu at (106.6, 90.8)
- added REF**: VIA_03_30mil, CustomFootprints:VIA_03_30mil, F.Cu at (112.5, 97.9)
- added REF**: VIA_03_30mil, CustomFootprints:VIA_03_30mil, F.Cu at (90.9, 115.6)
- added REF**: VIA_03_30mil, CustomFootprints:VIA_03_30mil, F.Cu at (87.2, 106.7)
- added REF**: VIA_03_30mil, CustomFootprints:VIA_03_30mil, F.Cu at (97.8, 108.5)
- added REF**: VIA_03_30mil, CustomFootprints:VIA_03_30mil, F.Cu at (90.9, 106.7)
- added REF**: VIA_03_30mil, CustomFootprints:VIA_03_30mil, F.Cu at (88.1, 116.5)
- added REF**: VIA_03_30mil, CustomFootprints:VIA_03_30mil, F.Cu at (90.9, 117.3)
- added REF**: VIA_03_30mil, CustomFootprints:VIA_03_30mil, F.Cu at (90.9, 113.8)
- added REF**: VIA_03_30mil, CustomFootprints:VIA_03_30mil, F.Cu at (90.9, 111.9)
- added REF**: VIA_03_30mil, CustomFootprints:VIA_03_30mil, F.Cu at (92.1, 120.8)
- added REF**: VIA_03_30mil, CustomFootprints:VIA_03_30mil, F.Cu at (92.1, 122.4)
- added REF**: VIA_03_30mil, CustomFootprints:VIA_03_30mil, F.Cu at (99.8, 116.2)
- added REF**: VIA_03_30mil, CustomFootprints:VIA_03_30mil, F.Cu at (99.8, 117.6)
- added REF**: VIA_03_30mil, CustomFootprints:VIA_03_30mil, F.Cu at (97.7, 117.6)
- added REF**: VIA_03_30mil, CustomFootprints:VIA_03_30mil, F.Cu at (100.1, 125.7)
- added REF**: VIA_03_30mil, CustomFootprints:VIA_03_30mil, F.Cu at (97.7, 119.3)
- added REF**: VIA_03_30mil, CustomFootprints:VIA_03_30mil, F.Cu at (105.7, 123.3)
- added REF**: VIA_03_30mil, CustomFootprints:VIA_03_30mil, F.Cu at (104.4, 123.3)
- added REF**: VIA_03_30mil, CustomFootprints:VIA_03_30mil, F.Cu at (103.1, 123.3)
- added REF**: VIA_03_30mil, CustomFootprints:VIA_03_30mil, F.Cu at (101.9, 123.3)
- added REF**: VIA_03_30mil, CustomFootprints:VIA_03_30mil, F.Cu at (105.7, 122.0)
- added REF**: VIA_03_30mil, CustomFootprints:VIA_03_30mil, F.Cu at (104.4, 122.0)
- added REF**: VIA_03_30mil, CustomFootprints:VIA_03_30mil, F.Cu at (103.1, 122.0)
- added REF**: VIA_03_30mil, CustomFootprints:VIA_03_30mil, F.Cu at (101.9, 122.0)
- added REF**: VIA_03_30mil, CustomFootprints:VIA_03_30mil, F.Cu at (105.7, 120.8)
- added REF**: VIA_03_30mil, CustomFootprints:VIA_03_30mil, F.Cu at (98.9, 126.1)
- added REF**: VIA_03_30mil, CustomFootprints:VIA_03_30mil, F.Cu at (104.4, 120.8)
- added REF**: VIA_03_30mil, CustomFootprints:VIA_03_30mil, F.Cu at (103.1, 120.8)
- added REF**: VIA_03_30mil, CustomFootprints:VIA_03_30mil, F.Cu at (101.9, 120.8)
- added REF**: VIA_03_30mil, CustomFootprints:VIA_03_30mil, F.Cu at (98.9, 125.1)
- added REF**: VIA_03_30mil, CustomFootprints:VIA_03_30mil, F.Cu at (92.2, 125.1)
- added REF**: VIA_03_30mil, CustomFootprints:VIA_03_30mil, F.Cu at (88.4, 124.5)
- added REF**: VIA_03_30mil, CustomFootprints:VIA_03_30mil, F.Cu at (87.1, 124.5)
- added REF**: VIA_03_30mil, CustomFootprints:VIA_03_30mil, F.Cu at (87.4, 131.6)
- added REF**: VIA_03_30mil, CustomFootprints:VIA_03_30mil, F.Cu at (109.7, 128.8)
- added REF**: VIA_03_30mil, CustomFootprints:VIA_03_30mil, F.Cu at (111.0, 127.5)
- added REF**: VIA_03_30mil, CustomFootprints:VIA_03_30mil, F.Cu at (96.6, 92.3)
- added REF**: VIA_03_30mil, CustomFootprints:VIA_03_30mil, F.Cu at (109.7, 126.2)
- added REF**: VIA_03_30mil, CustomFootprints:VIA_03_30mil, F.Cu at (97.3, 130.3)
- added REF**: VIA_03_30mil, CustomFootprints:VIA_03_30mil, F.Cu at (95.8, 130.3)
- added REF**: VIA_03_30mil, CustomFootprints:VIA_03_30mil, F.Cu at (94.2, 130.3)
- added REF**: VIA_03_30mil, CustomFootprints:VIA_03_30mil, F.Cu at (100.6, 129.2)
- added REF**: VIA_03_30mil, CustomFootprints:VIA_03_30mil, F.Cu at (104.9, 137.9)
- added REF**: VIA_03_30mil, CustomFootprints:VIA_03_30mil, F.Cu at (97.8, 137.9)
- added REF**: VIA_03_30mil, CustomFootprints:VIA_03_30mil, F.Cu at (90.2, 137.9)
- added REF**: VIA_03_30mil, CustomFootprints:VIA_03_30mil, F.Cu at (82.5, 137.9)
- added REF**: VIA_03_30mil, CustomFootprints:VIA_03_30mil, F.Cu at (82.5, 133.3)
- added REF**: VIA_03_30mil, CustomFootprints:VIA_03_30mil, F.Cu at (91.4, 92.3)
- added REF**: VIA_03_30mil, CustomFootprints:VIA_03_30mil, F.Cu at (113.8, 131.3)
- added REF**: VIA_03_30mil, CustomFootprints:VIA_03_30mil, F.Cu at (113.8, 127.5)
- added REF**: VIA_03_30mil, CustomFootprints:VIA_03_30mil, F.Cu at (113.8, 123.7)
- added REF**: VIA_03_30mil, CustomFootprints:VIA_03_30mil, F.Cu at (113.8, 116.1)
- added REF**: VIA_03_30mil, CustomFootprints:VIA_03_30mil, F.Cu at (112.1, 119.9)
- added REF**: VIA_03_30mil, CustomFootprints:VIA_03_30mil, F.Cu at (112.1, 116.1)
- added REF**: VIA_03_30mil, CustomFootprints:VIA_03_30mil, F.Cu at (113.8, 108.5)
- added REF**: VIA_03_30mil, CustomFootprints:VIA_03_30mil, F.Cu at (112.1, 112.3)
- added REF**: VIA_03_30mil, CustomFootprints:VIA_03_30mil, F.Cu at (111.9, 108.5)
- added REF**: VIA_03_30mil, CustomFootprints:VIA_03_30mil, F.Cu at (108.7, 112.0)
- added REF**: VIA_03_30mil, CustomFootprints:VIA_03_30mil, F.Cu at (87.1, 125.7)
- added REF**: VIA_03_30mil, CustomFootprints:VIA_03_30mil, F.Cu at (109.7, 113.3)
- added REF**: VIA_03_30mil, CustomFootprints:VIA_03_30mil, F.Cu at (108.0, 113.3)
- added REF**: VIA_03_30mil, CustomFootprints:VIA_03_30mil, F.Cu at (106.7, 112.0)
- added REF**: VIA_03_30mil, CustomFootprints:VIA_03_30mil, F.Cu at (105.4, 113.3)
- added REF**: VIA_03_30mil, CustomFootprints:VIA_03_30mil, F.Cu at (104.6, 108.5)
- added REF**: VIA_03_30mil, CustomFootprints:VIA_03_30mil, F.Cu at (113.8, 101.1)
- added REF**: VIA_03_30mil, CustomFootprints:VIA_03_30mil, F.Cu at (100.8, 108.5)
- added REF**: VIA_03_30mil, CustomFootprints:VIA_03_30mil, F.Cu at (112.5, 99.2)
- added REF**: VIA_03_30mil, CustomFootprints:VIA_03_30mil, F.Cu at (112.3, 105.2)
- added REF**: VIA_03_30mil, CustomFootprints:VIA_03_30mil, F.Cu at (108.7, 105.2)
- added REF**: VIA_03_30mil, CustomFootprints:VIA_03_30mil, F.Cu at (83.6, 120.7)
- added REF**: VIA_03_30mil, CustomFootprints:VIA_03_30mil, F.Cu at (104.6, 105.2)
- added REF**: VIA_03_30mil, CustomFootprints:VIA_03_30mil, F.Cu at (100.8, 105.2)
- added REF**: VIA_03_30mil, CustomFootprints:VIA_03_30mil, F.Cu at (97.0, 105.2)
- added REF**: VIA_03_30mil, CustomFootprints:VIA_03_30mil, F.Cu at (93.2, 105.2)
- C6: value 10uF -> 4,7uF
- moved C9 2.03 mm to (96.3, 125.2)
- moved R11 2.03 mm to (106.2, 130.8)
- moved R12 2.03 mm to (108.2, 130.8)
- moved R18 2.03 mm to (104.1, 130.8)
- moved R6 2.03 mm to (96.2, 120.9)
- moved R9 2.03 mm to (102.1, 130.8)
- moved U2 2.03 mm to (95.7, 127.8)
- moved C1 2.03 mm to (86.6, 119.6)
- moved C13 2.03 mm to (108.0, 115.5)
- moved C14 2.03 mm to (108.5, 127.5)
- moved C3 2.03 mm to (86.4, 121.4)
- moved C5 2.03 mm to (96.3, 122.4)
- moved C6 2.03 mm to (83.7, 116.6)
- moved C7 2.03 mm to (85.2, 116.6)
- moved D1 2.03 mm to (87.1, 111.8)
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Routing:
- net /LED1: track 29.0 -> 27.2 mm
- net /SW_USER: track 32.8 -> 31.2 mm
- net /OSC_IN: track 21.3 -> 19.8 mm
- net /IR_IN: track 43.7 -> 42.4 mm
- net /IR_CLK: track 30.7 -> 29.4 mm
- net /S_D+: track 7.40 -> 6.43 mm
- net /OSC_OUT: track 14.0 -> 14.9 mm
- net +3V3: track 147.2 -> 148.0 mm
Other:
- board size 37.3 x 52.1 mm -> 33.5 x 49.5 mm
- board text added: "SWD CLK"
- board text added: "SWD IO"
- board text removed: "SCLK"
- board text removed: "SIO"
