File: hardware/ir_converter.sch (KiCad schematic (older format))
At the start: 46 parts, among them J1 MX-47346-0001, J2 SWD, J3 TP, J4 TP, Q1 LL-S350PTC-1A, Q2 BC817-40, SW1 RESET, SW2 SW2, U1 TLV70033DDCT, U2 USBLC6-2, U3 STM32F103C8T6

Commit message: New PCB is ready.
Parts:
- added C11: 1uF, Capacitors_SMD:C_0603_HandSoldering, symbol C_Small
- C6: value 10uF -> 4,7uF
Connections:
- wire segments 129 -> 131
Changed lines of the file:
@@
 $EndComp
 $Comp
-L GND #PWR01
+L GND #PWR11
 U 1 1 58E4A14F
 P 1675 1525
-F 0 "#PWR01" H 1675 1275 50  0001 C CNN
+F 0 "#PWR11" H 1675 1275 50  0001 C CNN
 F 1 "GND" H 1675 1375 50  0000 C CNN
 F 2 "" H 1675 1525 50  0001 C CNN
@@
 $EndComp
 $Comp
-L GND #PWR02
+L GND #PWR15
 U 1 1 58E4A167
 P 2200 1450
-F 0 "#PWR02" H 2200 1200 50  0001 C CNN
+F 0 "#PWR15" H 2200 1200 50  0001 C CNN
 F 1 "GND" H 2200 1300 50  0000 C CNN
 F 2 "" H 2200 1450 50  0001 C CNN
@@
 P 2200 1325
 F 0 "C6" H 2210 1395 50  0000 L CNN
-F 1 "10uF" H 2210 1245 50  0000 L CNN
+F 1 "4,7uF" H 2210 1245 50  0000 L CNN
 F 2 "Capacitors_SMD:C_0603_HandSoldering" H 2200 1325 50  0001 C CNN
 F 3 "" H 2200 1325 50  0001 C CNN
@@
 $EndComp
 $Comp
-L GND #PWR03
+L GND #PWR2
 U 1 1 58E4A5C8
 P 600 1400
-F 0 "#PWR03" H 600 1150 50  0001 C CNN
+F 0 "#PWR2" H 600 1150 50  0001 C CNN
 F 1 "GND" H 600 1250 50  0000 C CNN
 F 2 "" H 600 1400 50  0001 C CNN
@@
 $EndComp
 $Comp
-L GND #PWR04
+L GND #PWR16
 U 1 1 58E4A63E
 P 2425 1450
-F 0 "#PWR04" H 2425 1200 50  0001 C CNN
+F 0 "#PWR16" H 2425 1200 50  0001 C CNN
 F 1 "GND" H 2425 1300 50  0000 C CNN
 F 2 "" H 2425 1450 50  0001 C CNN
@@
 $EndComp
 $Comp
-L +5V #PWR05
+L +5V #PWR1
 U 1 1 58E4A733
 P 600 1075
-F 0 "#PWR05" H 600 925 50  0001 C CNN
+F 0 "#PWR1" H 600 925 50  0001 C CNN
 F 1 "+5V" H 600 1215 50  0000 C CNN
 F 2 "" H 600 1075 50  0001 C CNN
@@
 $EndComp
 $Comp
-L +3.3V #PWR06
+L +3.3V #PWR17
 U 1 1 58E4A804
 P 2500 975
-F 0 "#PWR06" H 2500 825 50  0001 C CNN
+F 0 "#PWR17" H 2500 825 50  0001 C CNN
 F 1 "+3.3V" H 2500 1115 50  0000 C CNN
 F 2 "" H 2500 975 50  0001 C CNN
@@
 $EndComp
 $Comp
-L GND #PWR07
+L GND #PWR3
 U 1 1 58E4B22E
 P 850 3700
-F 0 "#PWR07" H 850 3450 50  0001 C CNN
+F 0 "#PWR3" H 850 3450 50  0001 C CNN
 F 1 "GND" H 850 3550 50  0000 C CNN
 F 2 "" H 850 3700 50  0001 C CNN
@@
 $EndComp
 $Comp
-L +5V #PWR08
+L +5V #PWR7
 U 1 1 58E4B4A3
 P 1150 2175
-F 0 "#PWR08" H 1150 2025 50  0001 C CNN
+F 0 "#PWR7" H 1150 2025 50  0001 C CNN
 F 1 "+5V" H 1150 2315 50  0000 C CNN
 F 2 "" H 1150 2175 50  0001 C CNN
@@
 U 1 1 58E4B595
 P 6600 975
-F 0 "C5" V 6775 875 50  0000 L CNN
-F 1 "100nF" V 6700 725 50  0000 L CNN
+F 0 "C5" H 6625 900 50  0000 L CNN
+F 1 "100nF" H 6600 1050 50  0000 L CNN
 F 2 "Capacitors_SMD:C_0603_HandSoldering" H 6600 975 50  0001 C CNN
 F 3 "" H 6600 975 50  0001 C CNN
@@
 $EndComp
 $Comp
-L GND #PWR09
+L GND #PWR10
 U 1 1 58E4B6CD
 P 1425 2250
-F 0 "#PWR09" H 1425 2000 50  0001 C CNN
+F 0 "#PWR10" H 1425 2000 50  0001 C CNN
 F 1 "GND" H 1425 2100 50  0000 C CNN
 F 2 "" H 1425 2250 50  0001 C CNN
@@
 $EndComp
 $Comp
-L GND #PWR010
+L GND #PWR31
 U 1 1 58E5740A
 P 7400 4975
-F 0 "#PWR010" H 7400 4725 50  0001 C CNN
+F 0 "#PWR31" H 7400 4725 50  0001 C CNN
 F 1 "GND" H 7400 4825 50  0000 C CNN
 F 2 "" H 7400 4975 50  0001 C CNN
@@
 $EndComp
 $Comp
-L PWR_FLAG #FLG011
+L PWR_FLAG #FLG1
 U 1 1 58E57AA9
 P 850 2250
-F 0 "#FLG011" H 850 2325 50  0001 C CNN
+F 0 "#FLG1" H 850 2325 50  0001 C CNN
 F 1 "PWR_FLAG" V 775 2375 50  0000 C CNN
 F 2 "" H 850 2250 50  0001 C CNN
@@
 $EndComp
 $Comp
-L PWR_FLAG #FLG012
+L PWR_FLAG #FLG3
 U 1 1 58E58086
 P 900 3675
-F 0 "#FLG012" H 900 3750 50  0001 C CNN
+F 0 "#FLG3" H 900 3750 50  0001 C CNN
 F 1 "PWR_FLAG" V 825 3875 50  0000 C CNN
 F 2 "" H 900 3675 50  0001 C CNN
@@
 $EndComp
 $Comp
-L +3.3V #PWR013
+L +3.3V #PWR30
 U 1 1 58E591A2
 P 7400 775
-F 0 "#PWR013" H 7400 625 50  0001 C CNN
+F 0 "#PWR30" H 7400 625 50  0001 C CNN
 F 1 "+3.3V" H 7400 915 50  0000 C CNN
 F 2 "" H 7400 775 50  0001 C CNN
@@
 $EndComp
 $Comp
-L GND #PWR014
+L GND #PWR29
 U 1 1 58E59A15
 P 7000 1200
-F 0 "#PWR014" H 7000 950 50  0001 C CNN
+F 0 "#PWR29" H 7000 950 50  0001 C CNN
 F 1 "GND" H 7000 1050 50  0000 C CNN
 F 2 "" H 7000 1200 50  0001 C CNN
@@
 $EndComp
 $Comp
-L GND #PWR015
+L GND #PWR6
 U 1 1 58E5AA95
 P 1075 7425
-F 0 "#PWR015" H 1075 7175 50  0001 C CNN
+F 0 "#PWR6" H 1075 7175 50  0001 C CNN
 F 1 "GND" H 1075 7275 50  0000 C CNN
 F 2 "" H 1075 7425 50  0001 C CNN
@@
 $EndComp
 $Comp
-L GND #PWR016
+L GND #PWR12
 U 1 1 58E5D294
 P 1700 7425
-F 0 "#PWR016" H 1700 7175 50  0001 C CNN
+F 0 "#PWR12" H 1700 7175 50  0001 C CNN
 F 1 "GND" H 1700 7275 50  0000 C CNN
 F 2 "" H 1700 7425 50  0001 C CNN
@@
 $EndComp
 $Comp
-L GND #PWR017
+L GND #PWR14
 U 1 1 58E5D761
 P 2000 7425
-F 0 "#PWR017" H 2000 7175 50  0001 C CNN
+F 0 "#PWR14" H 2000 7175 50  0001 C CNN
 F 1 "GND" H 2000 7275 50  0000 C CNN
 F 2 "" H 2000 7425 50  0001 C CNN
@@
 $EndComp
 $Comp
-L +3.3V #PWR018
+L +3.3V #PWR9
 U 1 1 58E5E7F1
 P 1325 2900
-F 0 "#PWR018" H 1325 2750 50  0001 C CNN
+F 0 "#PWR9" H 1325 2750 50  0001 C CNN
 F 1 "+3.3V" H 1325 3040 50  0000 C CNN
 F 2 "" H 1325 2900 50  0001 C CNN
@@
 $EndComp
 $Comp
-L GND #PWR019
+L GND #PWR5
 U 1 1 58E60729
 P 850 5850
-F 0 "#PWR019" H 850 5600 50  0001 C CNN
+F 0 "#PWR5" H 850 5600 50  0001 C CNN
 F 1 "GND" H 850 5700 50  0000 C CNN
 F 2 "" H 850 5850 50  0001 C CNN
@@
 $EndComp
 $Comp
-L +3.3V #PWR020
+L +3.3V #PWR18
 U 1 1 58E619F5
 P 2550 6625
-F 0 "#PWR020" H 2550 6475 50  0001 C CNN
+F 0 "#PWR18" H 2550 6475 50  0001 C CNN
 F 1 "+3.3V" H 2550 6765 50  0000 C CNN
 F 2 "" H 2550 6625 50  0001 C CNN
@@
 $EndComp
 $Comp
-L GND #PWR021
+L GND #PWR21
 U 1 1 58E62BB0
 P 2825 5950
-F 0 "#PWR021" H 2825 5700 50  0001 C CNN
+F 0 "#PWR21" H 2825 5700 50  0001 C CNN
 F 1 "GND" H 2825 5800 50  0000 C CNN
 F 2 "" H 2825 5950 50  0001 C CNN
@@
 $EndComp
 $Comp
-L +3.3V #PWR022
+L +3.3V #PWR20
 U 1 1 58E62E2A
 P 2625 5825
-F 0 "#PWR022" H 2625 5675 50  0001 C CNN
+F 0 "#PWR20" H 2625 5675 50  0001 C CNN
 F 1 "+3.3V" H 2625 5965 50  0000 C CNN
 F 2 "" H 2625 5825 50  0001 C CNN
@@
 $EndComp
 $Comp
-L GND #PWR023
+L GND #PWR26
 U 1 1 58E6782D
 P 5325 7510
-F 0 "#PWR023" H 5325 7260 50  0001 C CNN
+F 0 "#PWR26" H 5325 7260 50  0001 C CNN
 F 1 "GND" H 5325 7360 50  0000 C CNN
 F 2 "" H 5325 7510 50  0001 C CNN
@@
 $EndComp
 $Comp
-L GND #PWR024
+L GND #PWR28
 U 1 1 58E6994C
 P 6200 7500
-F 0 "#PWR024" H 6200 7250 50  0001 C CNN
+F 0 "#PWR28" H 6200 7250 50  0001 C CNN
 F 1 "GND" H 6200 7350 50  0000 C CNN
 F 2 "" H 6200 7500 50  0001 C CNN
@@
 $EndComp
 $Comp
-L +3.3V #PWR025
+L +3.3V #PWR27
 U 1 1 58E69F0E
 P 6200 6550
-F 0 "#PWR025" H 6200 6400 50  0001 C CNN
+F 0 "#PWR27" H 6200 6400 50  0001 C CNN
 F 1 "+3.3V" H 6200 6690 50  0000 C CNN
 F 2 "" H 6200 6550 50  0001 C CNN
@@
 $EndComp
 $Comp
-L GND #PWR026
+L GND #PWR8
 U 1 1 58E6D164
 P 1225 5850
-F 0 "#PWR026" H 1225 5600 50  0001 C CNN
+F 0 "#PWR8" H 1225 5600 50  0001 C CNN
 F 1 "GND" H 1225 5700 50  0000 C CNN
 F 2 "" H 1225 5850 50  0001 C CNN
@@
 $EndComp
 $Comp
-L +3.3V #PWR027
+L +3.3V #PWR4
 U 1 1 58E60893
 P 850 5250
-F 0 "#PWR027" H 850 5100 50  0001 C CNN
+F 0 "#PWR4" H 850 5100 50  0001 C CNN
 F 1 "+3.3V" H 850 5390 50  0000 C CNN
 F 2 "" H 850 5250 50  0001 C CNN
@@
 $EndComp
 $Comp
-L GND #PWR028
+L GND #PWR19
 U 1 1 58E71213
 P 2550 7575
-F 0 "#PWR028" H 2550 7325 50  0001 C CNN
+F 0 "#PWR19" H 2550 7325 50  0001 C CNN
 F 1 "GND" H 2550 7425 50  0000 C CNN
 F 2 "" H 2550 7575 50  0001 C CNN
@@
 $EndComp
 $Comp
-L GND #PWR029
+L GND #PWR23
 U 1 1 58E748BF
 P 3400 7550
-F 0 "#PWR029" H 3400 7300 50  0001 C CNN
+F 0 "#PWR23" H 3400 7300 50  0001 C CNN
 F 1 "GND" H 3400 7400 50  0000 C CNN
 F 2 "" H 3400 7550 50  0001 C CNN
@@
 $EndComp
 $Comp
-L +3.3V #PWR030
+L +3.3V #PWR22
 U 1 1 58E76017
 P 3400 6700
-F 0 "#PWR030" H 3400 6550 50  0001 C CNN
+F 0 "#PWR22" H 3400 6550 50  0001 C CNN
 F 1 "+3.3V" H 3400 6840 50  0000 C CNN
 F 2 "" H 3400 6700 50  0001 C CNN
@@
 $EndComp
 $Comp
-L GND #PWR031
+L GND #PWR13
 U 1 1 58E95985
 P 1850 3875
-F 0 "#PWR031" H 1850 3625 50  0001 C CNN
+F 0 "#PWR13" H 1850 3625 50  0001 C CNN
 F 1 "GND" H 1850 3725 50  0000 C CNN
 F 2 "" H 1850 3875 50  0001 C CNN
@@
 NoConn ~ 4600 4200
 $Comp
-L PWR_FLAG #FLG032
+L PWR_FLAG #FLG2
 U 1 1 58E7DF60
 P 850 2625
-F 0 "#FLG032" H 850 2700 50  0001 C CNN
+F 0 "#FLG2" H 850 2700 50  0001 C CNN
 F 1 "PWR_FLAG" V 775 2750 50  0000 C CNN
 F 2 "" H 850 2625 50  0001 C CNN
@@
 	2500 1125 2500 975
 Wire Wire Line
-	6600 825  7400 825
-Wire Wire Line
-	6600 1150 7125 1150
+	6175 825  7400 825
+Wire Wire Line
+	6175 1150 7125 1150
 Wire Wire Line
 	4600 3600 4100 3600
@@
 	4465 7220 4800 7220
 $Comp
-L +3.3V #PWR033
+L +3.3V #PWR25
 U 1 1 590A61E3
 P 5325 6195
-F 0 "#PWR033" H 5325 6045 50  0001 C CNN
+F 0 "#PWR25" H 5325 6045 50  0001 C CNN
 F 1 "+3.3V" H 5325 6335 50  0000 C CNN
 F 2 "" H 5325 6195 50  0001 C CNN
@@
 	4950 6500 4950 6475
 $Comp
-L GND #PWR034
+L GND #PWR24
 U 1 1 5924FDA3
 P 4950 6500
-F 0 "#PWR034" H 4950 6250 50  0001 C CNN
+F 0 "#PWR24" H 4950 6250 50  0001 C CNN
 F 1 "GND" H 4950 6350 50  0000 C CNN
 F 2 "" H 4950 6500 50  0001 C CNN
@@
 Text Label 1150 3300 0    60   ~ 0
 S_D-
+$Comp
+L C_Small C11
+U 1 1 5927ED52
+P 6175 975
+F 0 "C11" H 6185 1045 50  0000 L CNN
+F 1 "1uF" H 6185 895 50  0000 L CNN
+F 2 "Capacitors_SMD:C_0603_HandSoldering" H 6175 975 50  0001 C CNN
+F 3 "" H 6175 975 50  0001 C CNN
+	1    6175 975
+	1    0    0    -1
+$EndComp
+Wire Wire Line
+	6175 1075 6175 1150
+Connection ~ 6600 1150
+Wire Wire Line
+	6175 825  6175 875
+Connection ~ 6600 825
 $EndSCHEMATC
